File: MacPlusVGA.sch (KiCad schematic (older format))
At the start: 22 parts, among them J1 68000D, J2 DB15_Female_HighDensity, U1 M5LV-TQFP-144, U2 IS62C1024, U3 IS62C1024, U4 LD1117S33TR

Commit message: Board done? Needs some cleanup though
Parts:
- removed C13, C14, C15, C16: 2u2, stdpads:C_0603, symbol Device:C_Small
- removed J2: DB15_Female_HighDensity, Connector_Dsub:DSUB-15-HD_Female_Horizontal_P2.29x1.98mm_EdgePinOffset3.03mm_Housed_MountingHolesOffset4.94mm, symbol Connector:DB15_Female_HighDensity
- added J2: VGA, Connector_Dsub:DSUB-15-HD_Female_Horizontal_P2.29x1.98mm_EdgePinOffset3.03mm_Housed_MountingHolesOffset4.94mm, symbol Connector:DB15_Female_HighDensity_MountingHoles
- added J3: JTAG, stdpads:IDC_SMD_2x05_P2.54mm_Vertical, symbol Connector_Generic:Conn_02x05_Odd_Even
- added R1, R2, R3: 270, stdpads:R_0805, symbol Device:R_Small
- added R4, R5: 15, stdpads:R_0805, symbol Device:R_Small
- added U5: 25.175M, stdpads:Crystal_SMD_3225-4Pin_3.2x2.5mm, symbol GW_Logic:Oscillator_4P
- U4: footprint Package_TO_SOT_SMD:SOT-223-3_TabPin2 -> stdpads:SOT-223
Connections:
- net +3V3: now also J3.6 (Pin_6), U5.1 (EN), U5.4 (Vdd)
- net A1: now also U1.48 (IO34/1D4)
- net A10: now also U1.141 (IO102/0A6)
- net A11: now also U1.142 (IO103/0A7)
- net A12: now also U1.2 (IO0/0A8)
- net A13: now also U1.3 (IO1/0A9)
- net A14: now also U1.4 (IO2/0A10)
- net A15: now also U1.5 (IO3/0A11)
- net A16: now also U1.6 (IO4/0A12)
- net A17: now also U1.8 (IO5/0B13)
- net A18: now also U1.9 (IO6/0B12)
- net A19: now also U1.10 (IO7/0B11)
- net A2: now also U1.49 (IO35/1D7)
- net A20: now also U1.11 (IO8/0B8)
- net A21: now also U1.13 (IO9/0B5)
- net A22: now also U1.14 (IO10/0B4)
- net A23: now also U1.15 (IO11/0B3)
- net A3: now also U1.50 (IO36/1D8)
- net A4: now also U1.51 (IO37/1D11)
- net A5: now also U1.136 (IO97/0A1)
- net A6: now also U1.137 (IO98/0A2)
- net A7: now also U1.138 (IO99/0A3)
- net A8: now also U1.139 (IO100/0A4)
- net A9: now also U1.140 (IO101/0A5)
- net GND: now also C3.2, J2.0, J2.5, J2.6, J2.7, J2.8, J3.2 (Pin_2), J3.4 (Pin_4), U5.2 (GND)
- net RA1: now also U1.111 (IO78/3A7)
- net RA10: now also U1.121 (IO87/3D7)
- net RA11: now also U1.115 (IO82/3A3)
- net RA12: now also U1.119 (IO85/3D3)
- net RA13: now also U1.130 (IO92/0D11)
- net RA14: now also U1.129 (IO91/0D12)
- net RA15: now also U1.132 (IO94/0D7)
- net RA16: now also U1.134 (IO96/0D3)
- net RA17: now also U1.133 (IO95/0D4)
- net RA2: now also U1.112 (IO79/3A6)
- net RA3: now also U1.114 (IO81/3A4)
- net RA4: now also U1.116 (IO83/3A2)
- net RA5: now also U1.117 (IO84/3A1)
- net RA6: now also U1.120 (IO86/3D4)
- net RA7: now also U1.122 (IO88/3D8)
- net RA8: now also U1.124 (IO90/3D12)
- net RA9: now also U1.123 (IO89/3D11)
- net RD0: now also U1.98 (IO69/3B8)
- net RD1: now also U1.99 (IO70/3B11)
- net RD10: now also U1.103 (IO73/3A12)
- net RD11: now also U1.101 (IO72/3B13)
- net RD12: now also U1.104 (IO74/3A11)
- net RD13: now also U1.106 (IO76/3A9)
- net RD14: now also U1.96 (IO68/3B5)
- net RD15: now also U1.95 (IO67/3B4)
- net RD2: now also U1.100 (IO71/3B12)
- net RD3: now also U1.80 (IO57/2B13)
- net RD4: now also U1.81 (IO58/2B12)
- net RD5: now also U1.82 (IO59/2B11)
- net RD6: now also U1.85 (IO61/2B5)
- net RD7: now also U1.86 (IO62/2B4)
- net RD8: now also U1.107 (IO77/3A8)
- net RD9: now also U1.105 (IO75/3A10)
- net R~CS~H: now also U1.113 (IO80/3A5)
- net R~CS~L: now also U1.87 (IO63/2B3)
- net R~WE~: now also U1.131 (IO93/0D8)
- net TDI: now reaches U1.1 (TDI)
- net TDI: now also J3.5 (Pin_5)
- net TDO: now reaches U1.108 (TDO)
- net TDO: now also J3.7 (Pin_7)
- net TCK: now reaches U1.36 (TCK)
- net TCK: now also J3.1 (Pin_1)
- net B: now reaches U1.57 (IO39/2D12)
- net B: now also R3.2
- net G: now reaches U1.58 (IO40/2D11)
- net G: now also R2.2
- net R: now reaches U1.59 (IO41/2D8)
- net R: now also R1.2
- net HS: now reaches U1.60 (IO42/2D7)
- net HS: now also R4.1
- net VS: now reaches U1.61 (IO43/2D4)
- net VS: now also R5.1
- net TMS: now reaches U1.73 (TMS)
- net TMS: now also J3.3 (Pin_3)
- net at U1.92 (I1/CLK1): now also U5.3 (Output)
- new net Br: J2.3, R3.1
- new net Gr: J2.2, R2.1
- new net HSr: J2.13, R4.2
- new net Rr: J2.1, R1.1
- new net VSr: J2.14, R5.2
- no-connect marks 0 -> 28
Other:
- moved on the sheet: U2, U3

Commit message: As sent to JLCPCB July 2020
Parts:
- added C13, C14: 10u, stdpads:C_0805, symbol Device:C_Small
- J1: footprint Package_DIP:DIP-64_W22.86mm_LongPads -> stdpads:DIP-64-Slot
- U1: value M5LV-TQFP-144 -> M5LV-256/104-10VNC
Connections:
- net +5V: now also C13.1, C14.1
- net GND: now also J2.10, C13.2, C14.2
- no-connect marks 28 -> 27
Other:
- moved on the sheet: C1, C10, C11, C12, C2, C3, C4, C5, C6, C7, C8, C9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
