File: MacPlusVGA.kicad_pcb (KiCad board)
At the start: 2 copper layers, 84.3 x 60.2 mm, 23 parts, among them J1 68000D, J2 DB15_Female_HighDensity, U1 M5LV-TQFP-144, U2 IS62C1024, U3 IS62C1024, U4 LD1117S33TR

Commit message: Board done? Needs some cleanup though
Parts:
- removed C13, C14, C15, C16: 2u2, stdpads:C_0603
- removed REF**: Crystal_SMD_3225-4Pin_3.2x2.5mm, stdpads:Crystal_SMD_3225-4Pin_3.2x2.5mm
- added J3: IDC_SMD_2x05_P2.54mm_Vertical, stdpads:IDC_SMD_2x05_P2.54mm_Vertical, F.Cu at (209.2, 129.4)
- added R1: 270, stdpads:R_0805, F.Cu at (191.6, 131.8)
- added R2: 270, stdpads:R_0805, F.Cu at (189.6, 131.8)
- added R3: 270, stdpads:R_0805, F.Cu at (187.6, 131.8)
- added R4: 15, stdpads:R_0805, F.Cu at (193.6, 131.8)
- added R5: 15, stdpads:R_0805, F.Cu at (195.6, 131.8)
- added U5: 25.175M, stdpads:Crystal_SMD_3225-4Pin_3.2x2.5mm, F.Cu at (202.2, 115.2)
- C3, C4: value 2u2 -> 10u
- J2: value DB15_Female_HighDensity -> VGA
- U4: footprint Package_TO_SOT_SMD:SOT-223-3_TabPin2 -> stdpads:SOT-223
- moved C12 77.4 mm to (186.3, 102.3), turned to 180 degrees
- moved C11 65.3 mm to (186.3, 128.8)
- moved C10 53.0 mm to (195.3, 128.3)
- moved C9 51.3 mm to (199.1, 115.5), turned to 90 degrees
- moved C3 9.01 mm to (181.2, 68.7)
- moved C6 3.31 mm to (195.3, 102.8)
- moved J2 2.29 mm to (191.6, 136.1)
- moved C4 1.02 mm to (181.2, 85.5)
- moved U2 0.65 mm to (192.8, 74.4)
- moved U3 0.65 mm to (192.8, 91.2)
- moved C5 0.05 mm to (173.6, 115.5)
Connections:
- net Net-(U1-Pad108) renamed /TDO
- net Net-(U1-Pad73) renamed /TMS
- J2 pad 0: (no net) -> GND
- J2 pad 1: Net-(J2-Pad1) -> /Rr
- J2 pad 13: Net-(J2-Pad13) -> /HSr
- J2 pad 14: Net-(J2-Pad14) -> /VSr
- J2 pad 2: Net-(J2-Pad2) -> /Gr
- J2 pad 3: Net-(J2-Pad3) -> /Br
- J2 pad 5: Net-(J2-Pad5) -> GND
- J2 pad 6: Net-(J2-Pad6) -> GND
- J2 pad 7: Net-(J2-Pad7) -> GND
- J2 pad 8: Net-(J2-Pad8) -> GND
- U1 pad 1: /A11 -> /TDI
- U1 pad 100: Net-(U1-Pad100) -> /RD2
- U1 pad 101: Net-(U1-Pad101) -> /RD11
- U1 pad 103: Net-(U1-Pad103) -> /RD10
- U1 pad 104: Net-(U1-Pad104) -> /RD12
- U1 pad 105: Net-(U1-Pad105) -> /RD9
- U1 pad 106: Net-(U1-Pad106) -> /RD13
- U1 pad 107: Net-(U1-Pad107) -> /RD8
- U1 pad 111: Net-(U1-Pad111) -> /RA1
- U1 pad 112: Net-(U1-Pad112) -> /RA2
- U1 pad 113: Net-(U1-Pad113) -> /R~CS~H
- U1 pad 114: Net-(U1-Pad114) -> /RA3
- U1 pad 115: Net-(U1-Pad115) -> /RA11
- U1 pad 116: Net-(U1-Pad116) -> /RA4
- U1 pad 117: Net-(U1-Pad117) -> /RA5
- U1 pad 119: Net-(U1-Pad119) -> /RA12
- U1 pad 120: Net-(U1-Pad120) -> /RA6
- U1 pad 121: Net-(U1-Pad121) -> /RA10
- U1 pad 122: Net-(U1-Pad122) -> /RA7
- U1 pad 123: Net-(U1-Pad123) -> /RA9
- U1 pad 124: Net-(U1-Pad124) -> /RA8
- U1 pad 129: Net-(U1-Pad129) -> /RA14
- U1 pad 130: Net-(U1-Pad130) -> /RA13
- U1 pad 131: Net-(U1-Pad131) -> /R~WE~
- U1 pad 132: Net-(U1-Pad132) -> /RA15
- U1 pad 133: /A2 -> /RA17
- U1 pad 134: /A3 -> /RA16
- U1 pad 136: /A4 -> /A5
- U1 pad 137: /A5 -> /A6
- U1 pad 138: /A6 -> /A7
- U1 pad 139: /A7 -> /A8
- U1 pad 140: /A8 -> /A9
- U1 pad 141: /A9 -> /A10
- U1 pad 142: /A10 -> /A11
- U1 pad 23: /D15 -> /D14
- U1 pad 24: /D14 -> /D13
- U1 pad 26: /D13 -> /D12
- U1 pad 27: /D12 -> /D11
- U1 pad 28: /D11 -> /D10
- U1 pad 29: /D10 -> /D9
- U1 pad 31: /D9 -> /D8
- U1 pad 32: /D8 -> /D7
- U1 pad 33: /D7 -> /D6
- U1 pad 34: /D6 -> /D5
- U1 pad 35: /D5 -> /D4
- U1 pad 36: /D4 -> /TCK
- U1 pad 57: Net-(U1-Pad57) -> /B
- U1 pad 58: Net-(U1-Pad58) -> /G
- U1 pad 59: Net-(U1-Pad59) -> /R
- U1 pad 60: Net-(U1-Pad60) -> /HS
- U1 pad 61: Net-(U1-Pad61) -> /VS
- U1 pad 80: Net-(U1-Pad80) -> /RD3
- U1 pad 81: Net-(U1-Pad81) -> /RD4
- U1 pad 82: Net-(U1-Pad82) -> /RD5
- U1 pad 85: Net-(U1-Pad85) -> /RD6
- U1 pad 86: Net-(U1-Pad86) -> /RD7
- U1 pad 87: Net-(U1-Pad87) -> /R~CS~L
- U1 pad 95: Net-(U1-Pad95) -> /RD15
- U1 pad 96: Net-(U1-Pad96) -> /RD14
- U1 pad 98: Net-(U1-Pad98) -> /RD0
- U1 pad 99: Net-(U1-Pad99) -> /RD1
- U2 pad 13: /RD8 -> /RD0
- U2 pad 14: /RD9 -> /RD1
- U2 pad 15: /RD10 -> /RD2
- U3 pad 17: /RD3 -> /RD11
- U3 pad 18: /RD4 -> /RD12
- U3 pad 19: /RD5 -> /RD13
- U3 pad 20: /RD6 -> /RD14
- U3 pad 21: /RD7 -> /RD15
- U3 pad 22: /R~CS~L -> /R~CS~H
Routing:
- net +3V3: track 55.3 -> 239.9 mm, vias 38 -> 42
- net +5V: track 68.4 -> 222.7 mm, vias 14 -> 11
- net /RD15: track 0.00 -> 53.3 mm
- net /RD14: track 0.00 -> 50.9 mm
- net /TCK: track 0.00 -> 48.3 mm, vias 0 -> 2
- net /RD3: track 14.7 -> 62.0 mm
- net /RD4: track 14.7 -> 61.8 mm
- net /RD5: track 14.7 -> 61.6 mm
- net /RD6: track 14.7 -> 61.1 mm
- net /RD7: track 14.7 -> 61.0 mm
- net /R~CS~L: track 14.7 -> 61.0 mm
- net /RD0: track 0.00 -> 44.2 mm
- net /RD1: track 0.00 -> 41.6 mm
- net /RD2: track 0.00 -> 39.1 mm
- net /RD11: track 0.00 -> 28.7 mm
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- added copper zone on B.Cu, net +3V3
Other:
- board size 84.3 x 60.2 mm -> 130 x 77 mm
- net class Default: via_dia 0.5 -> 0.6; via_drill 0.2 -> 0.3
- rule via_min_drill: 0.2 -> 0.3
- rule via_min_size: 0.5 -> 0.6

Commit message: As sent to JLCPCB July 2020
Parts:
- added C13: 10u, stdpads:C_0805, F.Cu at (130.8, 113.2)
- added C14: 10u, stdpads:C_0805, F.Cu at (169.0, 113.2)
- J1: footprint Package_DIP:DIP-64_W22.86mm_LongPads -> stdpads:DIP-64-Slot
- J3: value IDC_SMD_2x05_P2.54mm_Vertical -> JTAG
- U1: value M5LV-TQFP-144 -> M5LV-256/104-10VNC
- moved J3 1.66 mm to (209.0, 131.1), turned to 180 degrees
- moved J1 0.13 mm to (86.4, 127.1)
Connections:
- J2 pad 10: Net-(J2-Pad10) -> GND
- J3 pad 1: (no net) -> /TCK
- J3 pad 10: (no net) -> Net-(J3-Pad10)
- J3 pad 2: (no net) -> GND
- J3 pad 3: (no net) -> /TMS
- J3 pad 4: (no net) -> GND
- J3 pad 5: (no net) -> /TDI
- J3 pad 6: (no net) -> +3V3
- J3 pad 7: (no net) -> /TDO
- J3 pad 8: (no net) -> Net-(J3-Pad8)
- J3 pad 9: (no net) -> Net-(J3-Pad9)
Routing:
- net +3V3: track 239.9 -> 474.9 mm, vias 42 -> 39
- net /TDI: track 9.67 -> 136.2 mm, vias 2 -> 4
- net GND: track 101.1 -> 128.4 mm, vias 218 -> 360
- net /TDO: track 12.5 -> 32.8 mm
- net /TMS: track 0.00 -> 19.7 mm
- net /TCK: track 48.3 -> 61.8 mm
- net +5V: track 222.7 -> 211.9 mm
- net /~LDS~: track 90.4 -> 88.8 mm
- added copper zone on F.Cu, net +3V3
- removed copper zone on B.Cu, net +3V3
Other:
- outline, holes or cut-outs redrawn
- rule solder_mask_min_width: 0.127 -> 0.1

Commit message: As sent to JLCPCB July 2020
Routing:
- net +3V3: track 474.9 -> 471.2 mm, vias 39 -> 19
- net GND: vias 360 -> 361
Changed lines of the file:
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@@
     (thickness 1.6)
     (drawings 16)
-    (tracks 1646)
+    (tracks 1626)
     (zones 0)
     (modules 27)
@@
   )
   (setup
-    (last_trace_width 0.15)
+    (last_trace_width 1)
     (user_trace_width 0.15)
     (user_trace_width 0.2)
@@
     (descr "15-pin D-Sub connector, horizontal/angled (90 deg), THT-mount, female, pitch 2.29x1.98mm, pin-PCB-offset 3.0300000000000002mm, distance of mounting holes 25mm, distance of mounting holes to PCB edge 4.9399999999999995mm, see https://disti-assets.s3.amazonaws.com/tonar/files/datasheets/16730.pdf")
     (tags "15-pin D-Sub connector horizontal angled 90deg THT female pitch 2.29x1.98mm pin-PCB-offset 3.0300000000000002mm mounting-holes-distance 25mm mounting-hole-offset 25mm")
-    (fp_text reference J2 (at -4.315 -2.61) (layer F.SilkS)
-      (effects (font (size 1 1) (thickness 0.15)))
+    (fp_text reference J2 (at -11.865 1.95) (layer F.SilkS)
+      (effects (font (size 0.8128 0.8128) (thickness 0.2032)))
     )
     (fp_text value VGA (at -4.315 14.89) (layer F.Fab)
@@
     (fp_line (start -1.6 1.25) (end 1.6 1.25) (layer F.Fab) (width 0.1))
     (fp_line (start -1.6 -1.25) (end -1.6 1.25) (layer F.Fab) (width 0.1))
-    (fp_text user %R (at 0 -2.25 90) (layer F.SilkS)
-      (effects (font (size 0.8128 0.8128) (thickness 0.2032)))
-    )
     (pad 4 smd roundrect (at -1.1 -0.85 90) (size 1.4 1.2) (layers F.Cu F.Paste F.Mask) (roundrect_rratio 0.25)
       (net 83 +3V3))
@@
   (via (at 122.555 106.426) (size 0.6) (drill 0.3) (layers F.Cu B.Cu) (net 2))
   (via (at 127.127 109.728) (size 0.6) (drill 0.3) (layers F.Cu B.Cu) (net 2))
+  (via (at 190.75 100.55) (size 0.6) (drill 0.3) (layers F.Cu B.Cu) (net 2))
   (segment (start 184.6 127.5) (end 184.6 126.2125) (width 0.15) (layer F.Cu) (net 3))
   (segment (start 182.7 130.6) (end 182.7 129.4) (width 0.15) (layer F.Cu) (net 3))
@@
   (segment (start 200.15 100.75) (end 198.501 99.101) (width 0.15) (layer F.Cu) (net 82))
   (segment (start 197.0125 107.3) (end 197.95 107.3) (width 0.15) (layer F.Cu) (net 82))
-  (via (at 178.1 101.75) (size 0.8) (drill 0.4) (layers F.Cu B.Cu) (net 83))
-  (segment (start 178.1 102.75) (end 178.1 101.75) (width 0.8) (layer F.Cu) (net 83))
   (segment (start 173.6 114.8) (end 174.35 114.8) (width 0.5) (layer F.Cu) (net 83))
   (segment (start 174.5 114.95) (end 174.5 115.2) (width 0.5) (layer F.Cu) (net 83))
   (segment (start 174.35 114.8) (end 174.5 114.95) (width 0.5) (layer F.Cu) (net 83))
   (segment (start 199.1 116.3) (end 198.35 116.3) (width 0.5) (layer F.Cu) (net 83))
-  (via (at 200.1 116.3) (size 0.8) (drill 0.4) (layers F.Cu B.Cu) (net 83))
   (segment (start 199.1 116.3) (end 200.1 116.3) (width 0.8) (layer F.Cu) (net 83))
   (segment (start 173.6 114.8) (end 172.6 114.8) (width 0.8) (layer F.Cu) (net 83))
-  (via (at 178.1 129.35) (size 0.8) (drill 0.4) (layers F.Cu B.Cu) (net 83))
-  (segment (start 178.1 128.35) (end 178.1 129.35) (width 0.8) (layer F.Cu) (net 83))
-  (via (at 178.1 103.7) (size 0.6) (drill 0.3) (layers F.Cu B.Cu) (net 83))
   (segment (start 178.1 104.8875) (end 178.1 103.7) (width 0.3) (layer F.Cu) (net 83))
   (segment (start 178.1 104.8875) (end 178.1 106.1) (width 0.3) (layer F.Cu) (net 83))
-  (via (at 194.6 103.7) (size 0.6) (drill 0.3) (layers F.Cu B.Cu) (net 83))
   (segment (start 194.6 104.8875) (end 194.6 103.7) (width 0.3) (layer F.Cu) (net 83))
   (segment (start 194.6 104.8875) (end 194.6 106.1) (width 0.3) (layer F.Cu) (net 83))
@@
   (segment (start 194.6 126.2125) (end 194.6 127.4) (width 0.3) (layer F.Cu) (net 83))
   (segment (start 178.1 126.2125) (end 178.1 125) (width 0.3) (layer F.Cu) (net 83))
-  (via (at 178.1 127.4) (size 0.6) (drill 0.3) (layers F.Cu B.Cu) (net 83))
   (segment (start 178.1 126.2125) (end 178.1 127.4) (width 0.3) (layer F.Cu) (net 83))
-  (via (at 122.8 114.55) (size 1) (drill 0.5) (layers F.Cu B.Cu) (net 83))
   (segment (start 124.45 114.55) (end 122.8 114.55) (width 1) (layer F.Cu) (net 83))
-  (via (at 126.1 114.55) (size 1) (drill 0.5) (layers F.Cu B.Cu) (net 83))
   (segment (start 124.45 114.55) (end 126.1 114.55) (width 1) (layer F.Cu) (net 83))
   (via (at 118.15 117.1) (size 1) (drill 0.5) (layers F.Cu B.Cu) (net 83))
   (segment (start 118.15 114.55) (end 118.15 117.1) (width 1) (layer F.Cu) (net 83))
   (segment (start 126.1 114.55) (end 127.45 114.55) (width 1) (layer F.Cu) (net 83))
-  (segment (start 194.6 102.75) (end 194.6 101.75) (width 0.8) (layer F.Cu) (net 83))
-  (via (at 193.75 102.75) (size 0.6) (drill 0.3) (layers F.Cu B.Cu) (net 83))
-  (segment (start 194.6 102.75) (end 193.75 102.75) (width 0.5) (layer F.Cu) (net 83))
-  (via (at 194.6 101.75) (size 0.8) (drill 0.4) (layers F.Cu B.Cu) (net 83))
   (segment (start 194.6 102.8) (end 194.6 103.7) (width 0.5) (layer F.Cu) (net 83))
-  (via (at 185.6 129.75) (size 0.8) (drill 0.4) (layers F.Cu B.Cu) (net 83))
-  (segment (start 185.6 128.75) (end 185.6 129.75) (width 0.8) (layer F.Cu) (net 83))
-  (segment (start 184.7 128.75) (end 184.65 128.8) (width 0.8) (layer F.Cu) (net 83))
-  (segment (start 185.6 128.75) (end 184.7 128.75) (width 0.8) (layer F.Cu) (net 83))
-  (via (at 184.65 128.8) (size 0.8) (drill 0.4) (layers F.Cu B.Cu) (net 83))
-  (via (at 187.95 102.35) (size 0.6) (drill 0.3) (layers F.Cu B.Cu) (net 83))
-  (segment (start 187.1 102.35) (end 187.95 102.35) (width 0.5) (layer F.Cu) (net 83))
-  (segment (start 187.1 102.35) (end 187.1 101.35) (width 0.8) (layer F.Cu) (net 83))
-  (via (at 187.1 101.35) (size 0.8) (drill 0.4) (layers F.Cu B.Cu) (net 83))
   (segment (start 185.6 115.55) (end 187.1 115.55) (width 0.5) (layer F.Cu) (net 83))
   (segment (start 185.6 115.2) (end 185.6 115.55) (width 0.5) (layer F.Cu) (net 83))
@@
   (segment (start 201.3 116.3) (end 200.1 116.3) (width 0.8) (layer F.Cu) (net 83))
   (segment (start 203 116.3) (end 201.3 116.3) (width 0.15) (layer F.Cu) (net 83))
-  (segment (start 187.1 126.2125) (end 187.1 127.5) (width 0.3) (layer F.Cu) (net 83))
-  (via (at 187.1 127.5) (size 0.6) (drill 0.3) (layers F.Cu B.Cu) (net 83))
   (segment (start 185.6 126.2125) (end 185.6 127.5) (width 0.3) (layer F.Cu) (net 83))
   (segment (start 185.6 127.5) (end 185.6 128.6) (width 0.5) (layer F.Cu) (net 83))
-  (via (at 185.6 127.5) (size 0.6) (drill 0.3) (layers F.Cu B.Cu) (net 83))
   (segment (start 194.6 128.35) (end 193.7 128.35) (width 0.5) (layer F.Cu) (net 83))
   (via (at 193.7 128.35) (size 0.6) (drill 0.3) (layers F.Cu B.Cu) (net 83))
@@
   (segment (start 176.75 115.3) (end 176.9 115.15) (width 0.3) (layer F.Cu) (net 83))
   (segment (start 175.6875 115.3) (end 176.75 115.3) (width 0.3) (layer F.Cu) (net 83))
-  (segment (start 178.1 102.75) (end 179 102.75) (width 0.5) (layer F.Cu) (net 83))
-  (via (at 179 102.75) (size 0.6) (drill 0.3) (layers F.Cu B.Cu) (net 83))
   (segment (start 185.6 106.2) (end 185.6 115.2) (width 0.5) (layer F.Cu) (net 83))
   (segment (start 185.6 104.8875) (end 185.6 106.2) (width 0.3) (layer F.Cu) (net 83))
   (segment (start 187.1 115.55) (end 187.1 106.2) (width 0.5) (layer F.Cu) (net 83))
   (segment (start 187.1 104.8875) (end 187.1 106.2) (width 0.3) (layer F.Cu) (net 83))
-  (segment (start 185.6 104.8875) (end 185.6 103.6) (width 0.3) (layer F.Cu) (net 83))
-  (via (at 185.6 103.6) (size 0.6) (drill 0.3) (layers F.Cu B.Cu) (net 83))
   (segment (start 187.1 104.8875) (end 187.1 103.6) (width 0.3) (layer F.Cu) (net 83))
-  (via (at 187.1 103.6) (size 0.6) (drill 0.3) (layers F.Cu B.Cu) (net 83))
   (segment (start 194.6 127.4) (end 194.6 128.35) (width 0.5) (layer F.Cu) (net 83))
   (segment (start 178.1 127.4) (end 178.1 128.35) (width 0.5) (layer F.Cu) (net 83))
@@
   (segment (start 198.2 116.15) (end 198.35 116.3) (width 0.5) (layer F.Cu) (net 83))
   (segment (start 198.2 115.95) (end 198.2 116.15) (width 0.5) (layer F.Cu) (net 83))
-  (segment (start 199.1 116.3) (end 199.1 117.2) (width 0.5) (layer F.Cu) (net 83))
-  (via (at 199.1 117.2) (size 0.6) (drill 0.3) (layers F.Cu B.Cu) (net 83))
   (segment (start 187.1 102.35) (end 187.1 103.6) (width 0.5) (layer F.Cu) (net 83))
   (segment (start 178.1 107.35) (end 194.6 107.35) (width 0.5) (layer F.Cu) (net 83))
@@
   (segment (start 118.15 117) (end 114.95 113.8) (width 1) (layer B.Cu) (net 83))
   (segment (start 118.15 117.1) (end 118.15 117) (width 1) (layer B.Cu) (net 83))
+  (segment (start 194.6 127.45) (end 193.7 128.35) (width 0.6) (layer B.Cu) (net 83))
+  (segment (start 194.6 127.4) (end 194.6 127.45) (width 0.6) (layer B.Cu) (net 83))
+  (segment (start 194.6 127.4) (end 194.6 128.35) (width 0.6) (layer B.Cu) (net 83))
+  (segment (start 194.6 127.4) (end 194.6 127.65) (width 0.6) (layer B.Cu) (net 83))
+  (segment (start 195.3 128.35) (end 195.5 128.35) (width 0.6) (layer B.Cu) (net 83))
+  (segment (start 194.6 127.65) (end 195.3 128.35) (width 0.6) (layer B.Cu) (net 83))
+  (segment (start 193.7 128.35) (end 193.95 128.1) (width 0.6) (layer B.Cu) (net 83))
+  (segment (start 193.7 128.35) (end 193.9 128.15) (width 0.6) (layer B.Cu) (net 83))
+  (segment (start 195.7 128.15) (end 196.342 127.508) (width 0.6) (layer B.Cu) (net 83))
+  (segment (start 193.9 128.15) (end 195.7 128.15) (width 0.6) (layer B.Cu) (net 83))
+  (segment (start 193.7 128.3) (end 193.7 128.35) (width 0.6) (layer B.Cu) (net 83))
+  (segment (start 194.6 127.4) (end 193.7 128.3) (width 0.6) (layer B.Cu) (net 83))
   (segment (start 197.8 114.8) (end 197.0125 114.8) (width 0.15) (layer F.Cu) (net 119))
   (segment (start 199.25 113.35) (end 197.8 114.8) (width 0.15) (layer F.Cu) (net 119))
